File: pcb/BleShield_teardrops_B2-16.brd (EAGLE design)
At the start: 23 parts, among them U1 ARDUINO_SHIELDNOHOLES, Y1 32.768KHz, 10 PPM

Commit message: re-did teardrops
Parts:
- moved U$7 6.61 mm to (43.0, 39.3)
- moved LED STRIP 0.58 mm to (9.82, 4.31)
Connections:
- net 5V: now also LED STRIP.4; no longer LED STRIP.1
- net GND: now also LED STRIP.1; no longer LED STRIP.4
- net MOSI: now also LED STRIP.2; no longer LED STRIP.3
- net SCK: now also LED STRIP.3; no longer LED STRIP.2
Routing:
- net 5V: track 75.4 -> 41.8 mm, vias 0 -> 2
- net GND: track 215.6 -> 219.6 mm, vias 5 -> 4
- net 3.3V: track 8.94 -> 12.6 mm
- net SCK: track 18.3 -> 21.7 mm
- net MOSI: track 22.6 -> 21.7 mm
