File: pcb/BleShield.brd (EAGLE design)
At the start: 53.3 x 48.3 mm, 30 parts, among them Q1 32.768K, 10ppm, SW1 SPST_TACT-EVQQ2, SW2 SPST_TACT-EVQQ2, U1 ARDUINO_SHIELDNOHOLES

Commit message: Update library name
Parts:
- Q1: device blinkiverse:CRYSTAL_3215 -> blinkinlabs:CRYSTAL_3215
- RGB_LED: device blinkiverse:LED-TRICOLOR-5050-FIXED -> blinkinlabs:LED-TRICOLOR-5050-FIXED
- U$7: device blinkiverse:OSHW-LOGO-L -> blinkinlabs:OSHW-LOGO-L
Changed lines of the file:
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@@
 <attribute name="NAME" x="41.5" y="11" size="0.6096" layer="25" align="bottom-right"/>
 </element>
-<element name="RGB_LED" library="blinkiverse" package="LED-TRICOLOR-5050-FIXED" value="LED-TRICOLOR-5050&quot;" x="23.5" y="7" smashed="yes" rot="R90">
+<element name="RGB_LED" library="blinkinlabs" package="LED-TRICOLOR-5050-FIXED" value="LED-TRICOLOR-5050&quot;" x="23.5" y="7" smashed="yes" rot="R90">
 <attribute name="VALUE" x="27.056" y="4.46" size="0.762" layer="27" rot="R90"/>
 </element>
-<element name="U$7" library="blinkiverse" package="OSHW-LOGO-L" value="" x="9.5" y="28"/>
+<element name="U$7" library="blinkinlabs" package="OSHW-LOGO-L" value="" x="9.5" y="28"/>
 <element name="LED1" library="adafruit" package="CHIPLED_0805" value="" x="44" y="45" smashed="yes" rot="R270">
 <attribute name="VALUE" x="42.73" y="42.46" size="1.27" layer="27"/>
@@
 <attribute name="VALUE" x="19.651" y="29.492" size="0.4064" layer="27" rot="R90"/>
 </element>
-<element name="Q1" library="blinkiverse" package="CRYSTAL_3215" value="32.768K, 10ppm" x="17.5" y="34" rot="R90"/>
+<element name="Q1" library="blinkinlabs" package="CRYSTAL_3215" value="32.768K, 10ppm" x="17.5" y="34" rot="R90"/>
 </elements>
 <signals>
